File: faceplates/C64 Pi1541-III Module FB1/C64 Pi1541-III Module FB1.kicad_pcb (KiCad board)
At the start: 2 copper layers, 100 x 100 mm, 7 parts, among them M1 Mounting, M2 Mounting, M3 Mounting, M4 Mounting

Commit message: Exported files
Parts:
- removed the REF** at (83.2, 56.5)
- removed REF***: KiCad-Logo2_6mm_SilkScreen, Symbols:KiCad-Logo2_6mm_SilkScreen
- added Pi1541-logo3: , Pi1541:Pi1541-logo3, B.Cu at (139.7, 79.4)
- added REF**: PWR_Spec, Pi1541:PWR_Specification_Single, B.Cu at (157.2, 56.5)
- added REF**: PWR_Spec, Pi1541:PWR_Specification_Single, F.Cu at (83.2, 56.5)
Other:
- board text removed: "Pi1541-III Faceplate FB1 github.com/tebl"
